File: kicad/column_board/column_driver.kicad_pcb (KiCad board)
At the start: 2 copper layers, 100 x 100 mm, 104 parts, among them J1 Panel column connector (femal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, J2 PWR_CHAIN_IN, J3 PWR_CHAIN_OUT, J4 DATA_CHAIN_IN, J5 DATA_CHAIN_OUT, U1 TPIC6B595, U10 TPIC6B595, U11 TPIC6B595, U12 TBD62783, U2 TPIC6B595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

Commit message: Add Gerber and DXF files for row and column boards
Parts:
- moved J5 22.1 mm to (30.0, 87.0)
- moved J4 22.0 mm to (30.0, 65.0)
Routing:
- net RC_DATA_OUT: track 102.5 -> 127.4 mm, vias 3 -> 4
- net RC_DATA: track 26.6 -> 48.5 mm
- net GND: track 125.8 -> 118.1 mm
- net RC_SHIFT_CLK: track 232.8 -> 238.2 mm, vias 3 -> 4
- net ~COL_EN: track 244.2 -> 248.3 mm, vias 3 -> 4
